File: kicad/4x4-buttoncell.kicad_pcb (KiCad board)
At the start: 2 copper layers, 90.3 x 77.6 mm, 64 parts, among them J1 Conn_01x02_Male, J2 Conn_01x04_Male, J3 Conn_01x03_Male, J4 Conn_01x06_Male, J5 Conn_01x02_Male, U1 STM32L031F4Px, U3 RFM9X

Commit message: gerber files V1 as sent to pcbway
Other:
- board size 90.3 x 77.6 mm -> 91.7 x 78.6 mm
- board text added: "+ - Cl Mo CS MI"
- board text added: "+ - TX"
- board text added: "- +"
- board text added: "Ant Gnd"
- board text added: "SCL SDA 3.3V + -"
- board text added: "SWC - SWD NR"
- board text added: "github.com/joba-1/STM32L0TTN.git"
