File: kicad/ST32ML011K4-Button.sch (KiCad schematic (older format))
At the start: 18 parts, among them J1 Conn_01x02_Male, J2 Conn_01x04_Male, J3 Conn_01x03_Male, J4 Conn_01x06_Male, J5 Conn_01x02_Male, U1 STM32L031F4Px, U3 RFM9X

Commit message: gerber files V1 as sent to pcbway
Connections:
- wire segments 15 -> 16
Other:
- moved on the sheet: C1, C2, D1, J1, J2, J3, J4, J5, R1, R2, R3, R4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
