File: kicad/ST32ML011K4-Button.kicad_pcb (KiCad board)
At the start: 2 copper layers, 90.3 x 77.6 mm, 64 parts, among them J1 Conn_01x02_Male, J2 Conn_01x04_Male, J3 Conn_01x03_Male, J4 Conn_01x06_Male, J5 Conn_01x02_Male, U1 STM32L031F4Px, U3 RFM9X

Commit message: undo autosave edits for 4x...
Parts:
- removed the C1 at (209.9, 85.9)
- removed the C1 at (209.6, 131.2)
- removed the C1 at (155.6, 131.4)
- removed the C2 at (208.7, 73.4)
- removed the C2 at (208.3, 118.7)
- removed the C2 at (154.3, 119.0)
- removed the D1 at (214.5, 73.3)
- removed the D1 at (214.1, 118.6)
- removed the D1 at (160.1, 118.9)
- removed the J1 at (202.9, 80.3)
- removed the J1 at (202.6, 125.6)
- removed the J1 at (148.6, 125.9)
- removed the J2 at (193.2, 93.3)
- removed the J2 at (192.8, 138.7)
- removed the J2 at (138.8, 138.9)
- removed the J3 at (191.0, 67.2)
- removed the J3 at (190.6, 112.5)
- removed the J3 at (136.7, 112.8)
- removed the J4 at (202.6, 67.2)
- removed the J4 at (202.2, 112.5)
- removed the J4 at (148.2, 112.8)
- removed the J5 at (207.5, 93.3)
- removed the J5 at (207.1, 138.7)
- removed the J5 at (153.2, 138.9)
- removed the R1 at (211.6, 73.3)
- removed the R1 at (211.2, 118.6)
- removed the R1 at (157.2, 118.9)
- removed the R2 at (214.4, 87.2)
- removed the R2 at (214.0, 132.6)
- removed the R2 at (160.0, 132.8)
- removed the TP1 at (188.3, 86.5)
- removed the TP1 at (188.0, 131.8)
- removed the TP1 at (134.0, 132.1)
- removed the TP2 at (188.5, 71.8)
- removed the TP2 at (188.1, 117.1)
- removed the TP2 at (134.1, 117.3)
- removed the TP3 at (188.5, 74.3)
- removed the TP3 at (188.1, 119.6)
- removed the TP3 at (134.1, 119.9)
- removed the TP4 at (188.3, 89.0)
- removed the TP4 at (188.0, 134.4)
- removed the TP4 at (134.0, 134.6)
- removed the U1 at (211.6, 80.1)
- removed the U1 at (211.2, 125.5)
- removed the U1 at (157.2, 125.7)
- removed the U3 at (198.4, 80.5)
- removed the U3 at (198.0, 125.9)
- removed the U3 at (144.0, 126.1)
Routing:
- net Net-(J5-Pad1): track 955.3 -> 238.8 mm, vias 12 -> 3
- net Earth: track 544.0 -> 136.0 mm, vias 24 -> 6
- net +3V3: track 354.8 -> 88.7 mm, vias 8 -> 2
- net NRESET: track 301.8 -> 75.4 mm
- net TX: track 147.5 -> 36.9 mm
- net TX_READY: track 138.9 -> 34.7 mm, vias 8 -> 2
- net SWDIO: track 136.0 -> 34.0 mm, vias 8 -> 2
- net RFM_CS: track 126.7 -> 31.7 mm, vias 8 -> 2
- net SWCLK: track 106.4 -> 26.6 mm, vias 4 -> 1
- net MISO: track 96.9 -> 24.2 mm
- net SCL: track 96.4 -> 24.1 mm, vias 4 -> 1
- net MOSI: track 96.0 -> 24.0 mm
- net SDA: track 93.3 -> 23.3 mm, vias 4 -> 1
- net SCK: track 85.1 -> 21.3 mm, vias 8 -> 2
- net RX_READY: track 77.4 -> 19.4 mm
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Other:
- board size 90.3 x 77.6 mm -> 37.6 x 32.9 mm
- board text added: "+ - Cl Mo CS MI"
- board text added: "+ - TX"
- board text added: "- +"
- board text added: "Ant Gnd"
- board text added: "SCL SDA 3.3V + -"
- board text added: "SWC - SWD NR"
- board text added: "github.com/joba-1/STM32L0TTN.git"
